File: pcb/qron0b.kicad_sch (KiCad schematic)
At the start: 32 parts, among them J1 ISP, SW1 SW_Right, U1 ATtiny24A-SS, U2 DS1302Z+, U3 74HC595, Y1 Crystal

Commit message: Update README
Other:
- title: Binary Watch -> qron0b
Changed lines of the file:
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@@
 	(paper "A4")
 	(title_block
-		(title "Binary Watch")
+		(title "qron0b")
 		(date "2025-01-14")
 		(rev "1")
